File: boards/crossover.sch (KiCad schematic (older format))
At the start: 47 parts, among them CON1 12VDC Power, J1 JACK_TRS_6PINS, P1 CONN_01X03, U1 TL074, U2 TL074, U4 TDA7292

Commit message: upadated boards
Parts:
- removed CON1: 12VDC Power, Connect:BARREL_JACK, symbol BARREL_JACK
- added C1, C2: 100n, Capacitors_ThroughHole:C_Disc_D3_P2.5, symbol C_Small
- added C25, C26, C27, C28: 100n, Capacitors_ThroughHole:C_Disc_D6_P5, symbol C_Small
- added R1: 100, Resistors_ThroughHole:Resistor_Horizontal_RM10mm, symbol R
- added RV?: DUAL_POT, symbol DUAL_POT
- added U? (x2): TL072, symbol TL072
- C10: renamed from C11; footprint Capacitors_SMD:C_0603_HandSoldering -> Capacitors_ThroughHole:C_Disc_D6_P5
- C11: renamed from C6; footprint Capacitors_SMD:C_0603_HandSoldering -> Capacitors_ThroughHole:C_Disc_D6_P5
- C12: footprint Capacitors_SMD:C_0603_HandSoldering -> Capacitors_ThroughHole:C_Disc_D6_P5
- C13: renamed from C7; footprint Capacitors_SMD:C_0603_HandSoldering -> Capacitors_ThroughHole:C_Disc_D3_P2.5
- C14: renamed from C8; footprint Capacitors_SMD:C_0603_HandSoldering -> Capacitors_ThroughHole:C_Disc_D3_P2.5
- C15: renamed from C13; footprint Capacitors_SMD:C_0603_HandSoldering -> Capacitors_ThroughHole:C_Disc_D3_P2.5
- C16: renamed from C14; footprint Capacitors_SMD:C_0603_HandSoldering -> Capacitors_ThroughHole:C_Disc_D3_P2.5
- C17: renamed from C15; footprint Capacitors_SMD:C_0603_HandSoldering -> Capacitors_ThroughHole:C_Disc_D6_P5
- C18: renamed from C16; footprint Capacitors_SMD:C_0603_HandSoldering -> Capacitors_ThroughHole:C_Disc_D6_P5
- C19: renamed from C17; value 200n -> 100n; footprint Capacitors_SMD:C_0603_HandSoldering -> Capacitors_ThroughHole:C_Disc_D6_P5
- C20: renamed from C18; value 200n -> 100n; footprint Capacitors_SMD:C_0603_HandSoldering -> Capacitors_ThroughHole:C_Disc_D6_P5
- C21: renamed from C19; footprint Capacitors_SMD:C_0603_HandSoldering -> Capacitors_ThroughHole:C_Disc_D6_P5
- C22: renamed from C20; footprint Capacitors_SMD:C_0603_HandSoldering -> Capacitors_ThroughHole:C_Disc_D6_P5
- C23: renamed from C21; footprint Capacitors_SMD:C_0603_HandSoldering -> Capacitors_ThroughHole:C_Disc_D6_P5
- C24: renamed from C22; footprint Capacitors_SMD:C_0603_HandSoldering -> Capacitors_ThroughHole:C_Disc_D6_P5
- C3: renamed from C1; value 220u -> 6800u; footprint Capacitors_ThroughHole:C_Radial_D10_L13_P5 -> Capacitors_ThroughHole:C_Radial_D16_L31.5_P7.5
- C4: renamed from C2; value 220u -> 6800u; footprint Capacitors_ThroughHole:C_Radial_D10_L13_P5 -> Capacitors_ThroughHole:C_Radial_D16_L31.5_P7.5
- C5: renamed from C3; footprint Capacitors_SMD:C_0603_HandSoldering -> Capacitors_ThroughHole:C_Disc_D6_P5
- C6: renamed from C9; footprint Capacitors_SMD:C_0603_HandSoldering -> Capacitors_ThroughHole:C_Disc_D6_P5
- C7: renamed from C4; value 200n -> 100n; footprint Capacitors_SMD:C_0603_HandSoldering -> Capacitors_ThroughHole:C_Disc_D6_P5
- C8: renamed from C10; value 200n -> 100n; footprint Capacitors_SMD:C_0603_HandSoldering -> Capacitors_ThroughHole:C_Disc_D6_P5
- C9: renamed from C5; footprint Capacitors_SMD:C_0603_HandSoldering -> Capacitors_ThroughHole:C_Disc_D6_P5
- D1: footprint (none) -> Diodes_ThroughHole:Diode_Bridge_15.7x15.7
- P1: value CONN_01X03 -> 12-0-12; footprint (none) -> Terminal_Blocks:TerminalBlock_Pheonix_MKDS1.5-3pol
- R10: renamed from R6; footprint Resistors_ThroughHole:Resistor_Horizontal_RM15mm -> Resistors_ThroughHole:Resistor_Horizontal_RM10mm
- R11: renamed from R10; footprint Resistors_ThroughHole:Resistor_Horizontal_RM15mm -> Resistors_ThroughHole:Resistor_Horizontal_RM10mm
- R12: renamed from R11; footprint Resistors_ThroughHole:Resistor_Horizontal_RM15mm -> Resistors_ThroughHole:Resistor_Horizontal_RM10mm
- R13: renamed from R12; footprint Resistors_ThroughHole:Resistor_Horizontal_RM15mm -> Resistors_ThroughHole:Resistor_Horizontal_RM10mm
- R14: renamed from R13; footprint Resistors_ThroughHole:Resistor_Horizontal_RM15mm -> Resistors_ThroughHole:Resistor_Horizontal_RM10mm
- R15: renamed from R14; footprint Resistors_ThroughHole:Resistor_Horizontal_RM15mm -> Resistors_ThroughHole:Resistor_Horizontal_RM10mm
- R16: renamed from R15; footprint Resistors_ThroughHole:Resistor_Horizontal_RM15mm -> Resistors_ThroughHole:Resistor_Horizontal_RM10mm
- R17: renamed from R16; footprint Resistors_ThroughHole:Resistor_Horizontal_RM15mm -> Resistors_ThroughHole:Resistor_Horizontal_RM10mm
- R18: renamed from R17; footprint Resistors_ThroughHole:Resistor_Horizontal_RM15mm -> Resistors_ThroughHole:Resistor_Horizontal_RM10mm
- R19: renamed from R18; footprint Resistors_ThroughHole:Resistor_Horizontal_RM15mm -> Resistors_ThroughHole:Resistor_Horizontal_RM10mm
- R2: renamed from R1; value 4K7 -> 1K 1W; footprint Resistors_ThroughHole:Resistor_Horizontal_RM15mm -> Resistors_ThroughHole:Resistor_Horizontal_RM10mm
- R3: renamed from R2; value 4K7 -> 1K 1W; footprint Resistors_ThroughHole:Resistor_Horizontal_RM15mm -> Resistors_ThroughHole:Resistor_Horizontal_RM10mm
- R4: renamed from R3; footprint Resistors_ThroughHole:Resistor_Horizontal_RM15mm -> Resistors_ThroughHole:Resistor_Horizontal_RM10mm
- R5: renamed from R7; footprint Resistors_ThroughHole:Resistor_Horizontal_RM15mm -> Resistors_ThroughHole:Resistor_Horizontal_RM10mm
- R6: renamed from R4; footprint Resistors_ThroughHole:Resistor_Horizontal_RM15mm -> Resistors_ThroughHole:Resistor_Horizontal_RM10mm
- R7: renamed from R8; footprint Resistors_ThroughHole:Resistor_Horizontal_RM15mm -> Resistors_ThroughHole:Resistor_Horizontal_RM10mm
- R8: renamed from R5; footprint Resistors_ThroughHole:Resistor_Horizontal_RM15mm -> Resistors_ThroughHole:Resistor_Horizontal_RM10mm
- R9: footprint Resistors_ThroughHole:Resistor_Horizontal_RM15mm -> Resistors_ThroughHole:Resistor_Horizontal_RM10mm
- renumbered U2 to U1, U1 to U2, U4 to U3
Connections:
- net labels added: +12V, -12V, GNDPWR
- net labels removed: +6V, -6V
- wire segments 107 -> 136
Other:
- note added: "Filter caps:\nhttps://www.digikey.com/product-detail/en/tdk-corporation/FG26C0G1H104JNT06/445-173396-1-ND/5812001"
- note added: "NPO, C0G for filter\nX7R for bypass"
- note added: "bypass caps:\nhttps://www.digikey.com/product-detail/en/kemet/C320C104K5R5TA7317/399-14036-1-ND/6562568"
- note added: "chasis ground"
- note added: "maybe higher power, need to up caps, etc."
- note removed: "Capacitors should be C0G (class 1)"
- note removed: "STA540..."
- note removed: "TDA2009 can be used\njust needs positive voltage + gnd\nmaybe switching supply with filter?"
- note removed: "TDA7496 = 5W+5W\nTDA2009 = 10W+10W (output through big capacitor, bad bass?)\nTDA7296= 14W+14W\nTDA7264 = 25W+25W (small num parts)\nTDA7292 = 40W+40W (lowest THD, better w/ dual supply, feedback resistors so you can control gain between tweeter & bass)"
- note removed: "if buffer input, could use general purp. op amp\nand just go op amp w/ virt grnd too..."
- note removed: "virtual ground: high output impedance power supply\ncan be lowered using op amp/buffer\nshould be ok, since only driving high impedance loads"
- moved on the sheet: C10, C11, C12, C13, C14, C15, C16, C17, C18, C19, C20, C21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

Commit message: some board work, added windows appveyor file
Parts:
- added T?: TRANSFO_3, symbol TRANSFO_3
- added U5: LM7815CT, TO_SOT_Packages_THT:TO-220_Neutral123_Vertical, symbol LM7815CT
- added U6: LM7915CT, TO_SOT_Packages_THT:TO-220_Neutral123_Vertical, symbol LM7915CT
- U4: renamed from U?; footprint (none) -> Housings_DIP:DIP-8_W7.62mm
- gave numbers to parts that had none: 1
Connections:
- wire segments 136 -> 137
Other:
- note added: "Design:\n10W in to each driver of a 8 ohm speaker\n-which means ~~9V and ~~1.1 A each\n-Power supply needs > 4.4 A, ~~5A\n-25W power dissipated in each chip\n\n1% THD\n-Vs needs +/- 22V\n-Transformer needs to be > 16-0-16, ~~5A (found 100VA, 20-0-20 on digikey)\n\nResevoir Caps\n- C = Q/V = I*t/V, I is ~~3 A, t = 1/60/2, V=allowed voltage drop = ~~4 V\n- C should be >6250u\n-put a small, better b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"
- note added: "supply voltage of tl074 is supposed to be 15 V, we're up at 28 now, might need regulator?"
Changed lines of the file:
@@
 bypass caps:\nhttps://www.digikey.com/product-detail/en/kemet/C320C104K5R5TA7317/399-14036-1-ND/6562568
 $Comp
-L -12V #PWR12
+L -12V #PWR9
 U 1 1 58E5C12B
 P 2550 3100
-F 0 "#PWR12" H 2550 3200 50  0001 C CNN
+F 0 "#PWR9" H 2550 3200 50  0001 C CNN
 F 1 "-12V" H 2550 3250 50  0000 C CNN
 F 2 "" H 2550 3100 50  0000 C CNN
@@
 $EndComp
 $Comp
-L -12V #PWR14
+L -12V #PWR11
 U 1 1 58E5C72F
 P 2550 5750
-F 0 "#PWR14" H 2550 5850 50  0001 C CNN
+F 0 "#PWR11" H 2550 5850 50  0001 C CNN
 F 1 "-12V" H 2550 5900 50  0000 C CNN
 F 2 "" H 2550 5750 50  0000 C CNN
@@
 	2750 850  2750 800
 $Comp
-L -12V #PWR5
+L -12V #PWR13
 U 1 1 58E5CC5E
 P 2750 1500
-F 0 "#PWR5" H 2750 1600 50  0001 C CNN
+F 0 "#PWR13" H 2750 1600 50  0001 C CNN
 F 1 "-12V" H 2750 1650 50  0000 C CNN
 F 2 "" H 2750 1500 50  0000 C CNN
@@
 maybe higher power, need to up caps, etc.
 $Comp
-L TL072 U?
+L TL072 U4
 U 1 1 58E6EA22
 P 3750 7300
-F 0 "U?" H 3750 7500 50  0000 L CNN
+F 0 "U4" H 3750 7500 50  0000 L CNN
 F 1 "TL072" H 3750 7100 50  0000 L CNN
-F 2 "" H 3750 7300 50  0000 C CNN
+F 2 "Housings_DIP:DIP-8_W7.62mm" H 3750 7300 50  0001 C CNN
 F 3 "" H 3750 7300 50  0000 C CNN
 	1    3750 7300
@@
 $EndComp
 $Comp
-L TL072 U?
+L TL072 U4
 U 2 1 58E6EAB3
 P 4450 7650
-F 0 "U?" H 4450 7850 50  0000 L CNN
+F 0 "U4" H 4450 7850 50  0000 L CNN
 F 1 "TL072" H 4450 7450 50  0000 L CNN
-F 2 "" H 4450 7650 50  0000 C CNN
+F 2 "Housings_DIP:DIP-8_W7.62mm" H 4450 7650 50  0001 C CNN
 F 3 "" H 4450 7650 50  0000 C CNN
 	2    4450 7650
@@
 $EndComp
 $Comp
-L DUAL_POT RV?
+L DUAL_POT RV1
 U 1 1 58E6EC42
 P 2850 7650
-F 0 "RV?" H 3010 7960 50  0000 C CNN
+F 0 "RV1" H 3010 7960 50  0000 C CNN
 F 1 "DUAL_POT" H 3140 7350 50  0000 C CNN
-F 2 "" H 2850 7650 50  0000 C CNN
+F 2 "" H 2850 7650 50  0001 C CNN
 F 3 "" H 2850 7650 50  0000 C CNN
 	1    2850 7650
 	1    0    0    -1
 $EndComp
+Text Notes 7650 1450 0    60   ~ 0
+Design:\n10W in to each driver of a 8 ohm speaker\n-which means ~~9V and ~~1.1 A each\n-Power supply needs > 4.4 A, ~~5A\n-25W power dissipated in each chip\n\n1% THD\n-Vs needs +/- 22V\n-Transformer needs to be > 16-0-16, ~~5A (found 100VA, 20-0-20 on digikey)\n\nResevoir Caps\n- C = Q/V = I*t/V, I is ~~3 A, t = 1/60/2, V=allowed voltage drop = ~~4 V\n- C should be >6250u\n-put a small, better behaved cap in parallel to decouple\n-put a resistor that discharges cap when power is off over 6.8 seconds (1k)
+Text Notes 4150 2250 0    60   ~ 0
+supply voltage of tl074 is supposed to be 15 V, we're up at 28 now, might need regulator?
+$Comp
+L LM7915CT U6
+U 1 1 58E7206A
+P 5350 1350
+F 0 "U6" H 5150 1150 50  0000 C CNN
+F 1 "LM7915CT" H 5350 1150 50  0000 L CNN
+F 2 "TO_SOT_Packages_THT:TO-220_Neutral123_Vertical" H 5350 1250 50  0000 C CIN
+F 3 "" H 5350 1350 50  0000 C CNN
+	1    5350 1350
+	1    0    0    -1
+$EndComp
+$Comp
+L LM7815CT U5
+U 1 1 58E72369
+P 4350 1300
+F 0 "U5" H 4150 1500 50  0000 C CNN
+F 1 "LM7815CT" H 4350 1500 50  0000 L CNN
+F 2 "TO_SOT_Packages_THT:TO-220_Neutral123_Vertical" H 4350 1400 50  0000 C CIN
+F 3 "" H 4350 1300 50  0000 C CNN
+	1    4350 1300
+	1    0    0    -1
+$EndComp
+Connection ~ 1550 5000
+Connection ~ 1550 4650
+Connection ~ 3750 5000
+Connection ~ 3750 4650
+Connection ~ 3750 2350
+Connection ~ 3750 2000
+$Comp
+L TRANSFO_3 T?
+U 1 1 58E73943
+P -900 1150
+F 0 "T?" H -900 1650 50  0000 C CNN
+F 1 "TRANSFO_3" H -900 650 50  0000 C CNN
+F 2 "" H -900 1150 50  0000 C CNN
+F 3 "" H -900 1150 50  0000 C CNN
+	1    -900 1150
+	1    0    0    -1
+$EndComp
+Wire Wire Line
+	-500 1050 -500 1250
 $EndSCHEMATC

Commit message: lots of updates, only trigger appveyor builds explicitly in commit message
Parts:
- R1: renamed from R2; footprint Resistors_ThroughHole:Resistor_Horizontal_RM10mm -> Resistors_ThroughHole:Resistor_Horizontal_RM15mm
- R2: renamed from R3; footprint Resistors_ThroughHole:Resistor_Horizontal_RM10mm -> Resistors_ThroughHole:Resistor_Horizontal_RM15mm
- gave numbers to parts that had none: 1
- renumbered C11 to C10, C23 to C11, C14 to C12, C5 to C13, C9 to C14, C17 to C15, C21 to C16, C8 to C17, C26 to C18, C15 to C19, C3 to C2, C28 to C21, C12 to C22, C24 to C23, C16 to C24, C6 to C25, C10 to C26, C18 to C27, C22 to C28, C2 to C3, C7 to C5, C25 to C6, C13 to C7, C19 to C8, C27 to C9, R18 to R10, R5 to R11, R9 to R12, R17 to R14, R7 to R15, R15 to R16, R11 to R17, R19 to R18, R1 to R19, R4 to R3, R8 to R4, R12 to R5, R16 to R6, R6 to R7, R14 to R8, R10 to R9, U5 to U1, U6 to U2, U1 to U3, U2 to U4, U3 to U5, U4 to U6
Other:
- moved on the sheet: RV1, U5A, U5B

Commit message: updates
Parts:
- removed U1: LM7815CT, TO_SOT_Packages_THT:TO-220_Neutral123_Vertical, symbol LM7815CT
- removed U2: LM7915CT, TO_SOT_Packages_THT:TO-220_Neutral123_Vertical, symbol LM7915CT
- added C3, C6: 100n, Capacitors_ThroughHole:C_Disc_D3_P2.5, symbol C_Small
- added R20, R21, R22, R23: RH, Resistors_ThroughHole:Resistor_Horizontal_RM10mm, symbol R
- R10: renamed from R9; value 2RH -> RH
- R11: renamed from R10; value 2RH -> RH
- R18: renamed from R17; value 2RH -> RH
- R19: renamed from R18; value 2RH -> RH
- RV1: footprint (none) -> Pin_Headers:Pin_Header_Straight_2x03
- renumbered C8 to C10, C9 to C11, C10 to C12, C11 to C13, C12 to C14, C13 to C15, C14 to C16, C15 to C17, C16 to C18, C17 to C19, C18 to C20, C19 to C21, C20 to C22, C21 to C23, C22 to C24, C23 to C25, C24 to C26, C25 to C27, C26 to C28, C27 to C29, C28 to C30, C3 to C4, C4 to C5, C5 to C7, C6 to C8, C7 to C9, R19 to R1, R11 to R12, R12 to R13, R13 to R14, R14 to R15, R15 to R16, R16 to R17, R1 to R2, R2 to R3, R3 to R4, R4 to R5, R5 to R6, R6 to R7, R7 to R8, R8 to R9, U6 to U1, U3 to U2, U4 to U2, U5 to U3, U3 to U4
Connections:
- wire segments 137 -> 173
Other:
- note added: "+/-12 V is actually more like 17 V (peak to peak)"
- note added: "Design:\n10W in to each 8 ohm driver\n-which means ~~9V and ~~1.1 A each\n-Power supply needs > 4.4 A, ~~5A\n- 20-25W power dissipated in each chip, 10W each driver = 80-90W\n\n1% THD\n-Vs needs +/- 20V (for 6 ohm, 13.5V)\n- 12-0-12 transformer will get ~~+/-17 V (maybe good enough)\n\nResevoir Caps\n- C = Q/V = I*t/V, I is ~~5 A, t = 1/60/2, \n- Supply V rejection ratio = 75 dB\ngain ~~30 dB, 75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"
- note added: "minimum gain 29 dB = 28x\navg. power = 1/2 V^2/R\nVpeak= 1V*G, with Vin-peak = 1 V\nwant 10 W output\nGain = sqrt(2*10* Rload)\n10 W per 8 ohm channel, given 1 Vpeak input, gain = 12.7 (too small?)"
- note removed: "Design:\n10W in to each driver of a 8 ohm speaker\n-which means ~~9V and ~~1.1 A each\n-Power supply needs > 4.4 A, ~~5A\n-25W power dissipated in each chip\n\n1% THD\n-Vs needs +/- 22V\n-Transformer needs to be > 16-0-16, ~~5A (found 100VA, 20-0-20 on digikey)\n\nResevoir Caps\n- C = Q/V = I*t/V, I is ~~3 A, t = 1/60/2, V=allowed voltage drop = ~~4 V\n- C should be >6250u\n-put a small, better b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"
- note removed: "maybe higher power, need to up caps, etc."
- note removed: "supply voltage of tl074 is supposed to be 15 V, we're up at 28 now, might need regulator?"
- moved on the sheet: J1, R1, RV1, U1A, U1B
