File: boards/amp/powersupply.sch (KiCad schematic (older format))
At the start: 105 parts, among them P1 CONN_01X03, P2 CONN_01X03, P3 CONN_01X04, P4 CONN_01X04, U1 TL072, U2 TL074, U3 TDA7292, U4 TL074, U5 TDA7292

Commit message: updated boards
Parts:
- removed C32: 1000u, Capacitors_ThroughHole:C_Radial_D10_L20_P5, symbol CP
- removed unit 2 of novalue3
- added D2: 6.8V, Diodes_ThroughHole:Diode_DO-35_SOD27_Horizontal_RM10, symbol D_Zener
- added novalue5: HEATSINK FOR TDA7292, symbol Heater
- added novalue6: POWER OUTLET, symbol LM317_SOT223
- added novalue7: fuse 1A, 250V rated, symbol LM317_SOT223
- D1: symbol Diode_Bridge -> D_Bridge_-A+A
- R10, R11, R12, R13, R14, R15, R16, R17, R18, R19, R20, R21, R22, R23, R4, R48, R49, R5, R50, R51, R6, R7, R8, R9: footprint Resistors_ThroughHole:Resistor_Horizontal_RM7mm -> scimpy_library:R_Axial_DIN0204_L3.6mm_D1.6mm_P5.08mm_Horizontal
- R24, R25, R26, R27, R28, R29, R30, R31, R32, R33, R34, R35: footprint Resistors_ThroughHole:Resistor_Horizontal_RM10mm -> scimpy_library:R_Axial_DIN0204_L3.6mm_D1.6mm_P5.08mm_Horizontal
- R36: value 1K -> 18K; footprint Resistors_ThroughHole:Resistor_Horizontal_RM7mm -> scimpy_library:R_Axial_DIN0204_L3.6mm_D1.6mm_P5.08mm_Horizontal; manf# CFR16J1K0 -> (none)
- RV1, novalue1, novalue2: symbol DUAL_POT -> POT_Dual
- novalue3: footprint TO_SOT_Packages_THT:Multiwatt-11_Vertical_StaggeredType1 -> (none); symbol TDA7292 -> Heater
- novalue4: symbol TRANSFO_3 -> Transformer_SP_2S
Connections:
- net labels added: Vs-6.8V
- net labels removed: 1s_delay
Other:
- note added: "make modular:\npower supply\nvolume + BS/buffer + phase (cab parameters)\nxover (driver parameters)\namp"
