File: boards/amp/amp.kicad_pcb (KiCad board)
At the start: 2 copper layers, 104.1 x 51.8 mm, 51 parts, among them P1 CONN_01X04, P2 CONN_01X07, P3 CONN_01X03, P4 CONN_01X04, Q1 BC107, SW1 Standby, SW2 Mute, U1 TDA7292, U2 TDA7292

Commit message: more boards work
Routing:
- added copper zone on B.Cu, net GND
- added copper zone on F.Cu, net GND
