File: boards/amp/amp.sch (KiCad schematic (older format))
At the start: 47 parts, among them P1 CONN_01X04, P2 CONN_01X07, P3 CONN_01X03, P4 CONN_01X04, Q1 BC107, SW1 Standby, SW2 Mute, U1 TDA7292, U2 TDA7292

Commit message: more boards work
Parts:
- added novalue3: Standby-switch, symbol SW_SPDT
- added novalue4: Mute-switch, symbol SW_SPST
- added novalue5: wire2con, symbol SW_SPST
- added novalue6: wire2con, symbol SW_SPDT
- added novalue7: Amp-Enclosure, symbol Speaker
- added novalue8: Amp-Enclosure-Cover, symbol Speaker
- C2: manf# (none) -> K104K15X7RF53L2
- C3: manf# (none) -> 105CKR050M
- P2: manf# (none) -> 0022286070
- P3: manf# (none) -> 1935174
- R1, R13: manf# (none) -> LR0204F10K
- R10: manf# (none) -> MCMF0W4FF1502A50
- R12, R5, R8: value 4.8R -> 4.7R
- R16: manf# (none) -> MCMF0W4FF4702A50
- R2: value 4.8R -> 4.7R; manf# (none) -> MCCFR0W4J047JA50
- R3: manf# (none) -> LR0204F560R
- R4: manf# (none) -> MCMF0W4FF6802A50
- R6: manf# (none) -> MCMF0W4FF1501A50
- SW1, SW2: manf# (none) -> 640456-2
Changed lines of the file:
@@
 F 2 "scimpy_library:R_Axial_DIN0204_L3.6mm_D1.6mm_P5.08mm_Horizontal" V 5730 2900 50  0001 C CNN
 F 3 "" H 5800 2900 50  0000 C CNN
+F 4 "MCMF0W4FF6802A50" V 5800 2900 60  0001 C CNN "manf#"
 	1    5800 2900
 	-1   0    0    1
@@
 F 2 "scimpy_library:R_Axial_DIN0204_L3.6mm_D1.6mm_P5.08mm_Horizontal" V 5730 3500 50  0001 C CNN
 F 3 "" H 5800 3500 50  0000 C CNN
+F 4 "MCMF0W4FF1501A50" V 5800 3500 60  0001 C CNN "manf#"
 	1    5800 3500
 	-1   0    0    1
@@
 P 6150 3000
 F 0 "R5" V 6230 3000 50  0000 C CNN
-F 1 "4.8R" V 6150 3000 50  0000 C CNN
+F 1 "4.7R" V 6150 3000 50  0000 C CNN
 F 2 "scimpy_library:R_Axial_DIN0204_L3.6mm_D1.6mm_P5.08mm_Horizontal" V 6080 3000 50  0001 C CNN
 F 3 "" H 6150 3000 50  0000 C CNN
@@
 F 2 "scimpy_library:R_Axial_DIN0204_L3.6mm_D1.6mm_P5.08mm_Horizontal" V 6130 1700 50  0001 C CNN
 F 3 "" H 6200 1700 50  0000 C CNN
+F 4 "MCMF0W4FF1802A50" V 6200 1700 60  0001 C CNN "manf#"
+F 5 "LR0204F10K" V 6200 1700 60  0001 C CNN "manf#"
 	1    6200 1700
 	-1   0    0    1
@@
 P 6550 1700
 F 0 "R2" V 6630 1700 50  0000 C CNN
-F 1 "4.8R" V 6550 1700 50  0000 C CNN
+F 1 "4.7R" V 6550 1700 50  0000 C CNN
 F 2 "scimpy_library:R_Axial_DIN0204_L3.6mm_D1.6mm_P5.08mm_Horizontal" V 6480 1700 50  0001 C CNN
 F 3 "" H 6550 1700 50  0000 C CNN
+F 4 "MCCFR0W4J047JA50" V 6550 1700 60  0001 C CNN "manf#"
 	1    6550 1700
 	-1   0    0    1
@@
 F 2 "Capacitors_ThroughHole:C_Disc_D3_P2.5" H 6550 2050 50  0001 C CNN
 F 3 "" H 6550 2050 50  0000 C CNN
+F 4 "K104K15X7RF53L2" H 6550 2050 60  0001 C CNN "manf#"
 	1    6550 2050
 	1    0    0    -1
@@
 P 5700 6400
 F 0 "R12" V 5780 6400 50  0000 C CNN
-F 1 "4.8R" V 5700 6400 50  0000 C CNN
+F 1 "4.7R" V 5700 6400 50  0000 C CNN
 F 2 "scimpy_library:R_Axial_DIN0204_L3.6mm_D1.6mm_P5.08mm_Horizontal" V 5630 6400 50  0001 C CNN
 F 3 "" H 5700 6400 50  0000 C CNN
@@
 P 6150 4650
 F 0 "R8" V 6230 4650 50  0000 C CNN
-F 1 "4.8R" V 6150 4650 50  0000 C CNN
+F 1 "4.7R" V 6150 4650 50  0000 C CNN
 F 2 "scimpy_library:R_Axial_DIN0204_L3.6mm_D1.6mm_P5.08mm_Horizontal" V 6080 4650 50  0001 C CNN
 F 3 "" H 6150 4650 50  0000 C CNN
@@
 F 2 "scimpy_library:R_Axial_DIN0204_L3.6mm_D1.6mm_P5.08mm_Horizontal" V 6130 2100 50  0001 C CNN
 F 3 "" H 6200 2100 50  0000 C CNN
+F 4 "LR0204F560R" V 6200 2100 60  0001 C CNN "manf#"
 	1    6200 2100
 	-1   0    0    1
@@
 F 2 "Pin_Headers:Pin_Header_Angled_1x07" H 1450 3150 50  0001 C CNN
 F 3 "" H 1450 3150 50  0000 C CNN
+F 4 "0022286070" H 1450 3150 60  0001 C CNN "manf#"
 	1    1450 3150
 	-1   0    0    1
@@
 F 2 "Capacitors_ThroughHole:C_Radial_D10_L20_P5" H 5638 2100 50  0001 C CNN
 F 3 "" H 5600 2250 50  0000 C CNN
+F 4 "105CKR050M" H 5600 2250 60  0001 C CNN "manf#"
 	1    5600 2250
 	1    0    0    -1
@@
 F 2 "Terminal_Blocks:TerminalBlock_Pheonix_MKDS1.5-3pol" H 1650 4700 50  0001 C CNN
 F 3 "" H 1650 4700 50  0000 C CNN
+F 4 "1935174" H 1650 4700 60  0001 C CNN "manf#"
 	1    1650 4700
 	-1   0    0    -1
@@
 F 2 "scimpy_library:R_Axial_DIN0204_L3.6mm_D1.6mm_P5.08mm_Horizontal" V 1480 5850 50  0001 C CNN
 F 3 "" H 1550 5850 50  0000 C CNN
+F 4 "MCMF0W4FF1502A50" V 1550 5850 60  0001 C CNN "manf#"
 	1    1550 5850
 	-1   0    0    1
@@
 F 2 "scimpy_library:R_Axial_DIN0204_L3.6mm_D1.6mm_P5.08mm_Horizontal" V 2580 7100 50  0001 C CNN
 F 3 "" H 2650 7100 50  0000 C CNN
+F 4 "MCMF0W4FF4702A50" V 2650 7100 60  0001 C CNN "manf#"
 	1    2650 7100
 	-1   0    0    1
@@
 F 2 "scimpy_library:R_Axial_DIN0204_L3.6mm_D1.6mm_P5.08mm_Horizontal" V 1580 6500 50  0001 C CNN
 F 3 "" H 1650 6500 50  0000 C CNN
+F 4 "LR0204F10K" V 1650 6500 60  0001 C CNN "manf#"
 	1    1650 6500
 	0    -1   -1   0
@@
 F 2 "Connectors_Molex:Molex_KK-6410-03_03x2.54mm_Straight" H 1300 6500 50  0001 C CNN
 F 3 "" H 1300 6500 50  0000 C CNN
+F 4 "640456-2" H 1300 6500 60  0001 C CNN "manf#"
 	1    1300 6500
 	-1   0    0    1
@@
 F 2 "Connectors_Molex:Molex_KK-6410-02_02x2.54mm_Straight" H 2400 7450 50  0001 C CNN
 F 3 "" H 2400 7450 50  0000 C CNN
+F 4 "640456-2" H 2400 7450 60  0001 C CNN "manf#"
 	1    2400 7450
 	0    -1   -1   0
@@
 Text Notes 8400 5850 0    60   ~ 0
 route all first, then do pours to make sure ground gets good thicknesses
+$Comp
+L SW_SPDT novalue3
+U 1 1 5930858D
+P 1350 7300
+F 0 "novalue3" H 1350 7470 50  0000 C CNN
+F 1 "Standby-switch" H 1350 7100 50  0000 C CNN
+F 2 "" H 1350 7300 50  0001 C CNN
+F 3 "" H 1350 7300 50  0000 C CNN
+F 4 "SRJ23A3BBBNN" H 1350 7300 60  0001 C CNN "manf#"
+	1    1350 7300
+	-1   0    0    1
+$EndComp
+$Comp
+L SW_SPST novalue4
+U 1 1 593086FB
+P 2950 7450
+F 0 "novalue4" H 2950 7575 50  0000 C CNN
+F 1 "Mute-switch" H 2950 7350 50  0000 C CNN
+F 2 "" H 2950 7450 50  0001 C CNN
+F 3 "" H 2950 7450 50  0000 C CNN
+F 4 "R13-23B-05-BW" H 2950 7450 60  0001 C CNN "manf#"
+	1    2950 7450
+	0    -1   -1   0
+$EndComp
+$Comp
+L SW_SPDT novalue6
+U 1 1 593096EE
+P 1350 7850
+F 0 "novalue6" H 1350 8020 50  0000 C CNN
+F 1 "wire2con" H 1350 7650 50  0000 C CNN
+F 2 "" H 1350 7850 50  0001 C CNN
+F 3 "" H 1350 7850 50  0000 C CNN
+F 4 "3-640440-2" H 1350 7850 60  0001 C CNN "manf#"
+	1    1350 7850
+	-1   0    0    1
+$EndComp
+$Comp
+L SW_SPST novalue5
+U 1 1 5930991C
+P 3350 7450
+F 0 "novalue5" H 3350 7575 50  0000 C CNN
+F 1 "wire2con" H 3350 7350 50  0000 C CNN
+F 2 "" H 3350 7450 50  0001 C CNN
+F 3 "" H 3350 7450 50  0000 C CNN
+F 4 "3-640440-2" H 3350 7450 60  0001 C CNN "manf#"
+	1    3350 7450
+	0    -1   -1   0
+$EndComp
+$Comp
+L Speaker novalue7
+U 1 1 59317D4C
+P 9650 1050
+F 0 "novalue7" H 9700 1275 50  0000 R CNN
+F 1 "Amp-Enclosure" H 9700 1200 50  0000 R CNN
+F 2 "" H 9650 850 50  0000 C CNN
+F 3 "" H 9640 1000 50  0000 C CNN
+F 4 "AC-404" H 9650 1050 60  0001 C CNN "manf#"
+	1    9650 1050
+	1    0    0    -1
+$EndComp
+$Comp
+L Speaker novalue8
+U 1 1 59318089
+P 9650 1600
+F 0 "novalue8" H 9700 1825 50  0000 R CNN
+F 1 "Amp-Enclosure-Cover" H 9700 1750 50  0000 R CNN
+F 2 "" H 9650 1400 50  0000 C CNN
+F 3 "" H 9640 1550 50  0000 C CNN
+F 4 "BPA-1591" H 9650 1600 60  0001 C CNN "manf#"
+	1    9650 1600
+	1    0    0    -1
+$EndComp
 $EndSCHEMATC
