File: boards/powersupply/phase.sch (KiCad schematic (older format))
At the start: 19 parts, among them U6 TL074

Commit message: updated boards
Parts:
- R1, R37, R38, R39, R40, R41, R42, R43, R44, R45, R46, R47: footprint Resistors_ThroughHole:Resistor_Horizontal_RM7mm -> scimpy_library:R_Axial_DIN0204_L3.6mm_D1.6mm_P5.08mm_Horizontal
- U6: footprint (none) -> Housings_DIP:DIP-14_W7.62mm
Changed lines of the file:
@@
 LIBS:tda7292
 LIBS:audio
-LIBS:crossover-cache
 EELAYER 25 0
 EELAYER END
@@
 $EndComp
 $Comp
-L +12V #PWR52
+L +12V #PWR046
 U 1 1 5900A021
 P 3900 1450
-F 0 "#PWR52" H 3900 1300 50  0001 C CNN
+F 0 "#PWR046" H 3900 1300 50  0001 C CNN
 F 1 "+12V" H 3900 1590 50  0000 C CNN
 F 2 "" H 3900 1450 50  0000 C CNN
@@
 $EndComp
 $Comp
-L GND #PWR57
+L GND #PWR047
 U 1 1 58FFF572
 P 4100 2700
-F 0 "#PWR57" H 4100 2450 50  0001 C CNN
+F 0 "#PWR047" H 4100 2450 50  0001 C CNN
 F 1 "GND" H 4100 2550 50  0000 C CNN
 F 2 "" H 4100 2700 50  0000 C CNN
@@
 F 0 "R38" V 3630 2300 50  0000 C CNN
 F 1 "Rph" V 3550 2300 50  0000 C CNN
-F 2 "Resistors_ThroughHole:Resistor_Horizontal_RM7mm" V 3480 2300 50  0001 C CNN
+F 2 "scimpy_library:R_Axial_DIN0204_L3.6mm_D1.6mm_P5.08mm_Horizontal" V 3480 2300 50  0001 C CNN
 F 3 "" H 3550 2300 50  0000 C CNN
 	1    3550 2300
@@
 $EndComp
 $Comp
-L GND #PWR55
+L GND #PWR048
 U 1 1 58FFFCE8
 P 3550 2450
-F 0 "#PWR55" H 3550 2200 50  0001 C CNN
+F 0 "#PWR048" H 3550 2200 50  0001 C CNN
 F 1 "GND" H 3550 2300 50  0000 C CNN
 F 2 "" H 3550 2450 50  0000 C CNN
@@
 F 0 "R1" V 3430 1250 50  0000 C CNN
 F 1 "2K2" V 3350 1250 50  0000 C CNN
-F 2 "Resistors_ThroughHole:Resistor_Horizontal_RM7mm" V 3280 1250 50  0001 C CNN
+F 2 "scimpy_library:R_Axial_DIN0204_L3.6mm_D1.6mm_P5.08mm_Horizontal" V 3280 1250 50  0001 C CNN
 F 3 "" H 3350 1250 50  0000 C CNN
 	1    3350 1250
@@
 F 0 "R37" V 4280 1250 50  0000 C CNN
 F 1 "2K2" V 4200 1250 50  0000 C CNN
-F 2 "Resistors_ThroughHole:Resistor_Horizontal_RM7mm" V 4130 1250 50  0001 C CNN
+F 2 "scimpy_library:R_Axial_DIN0204_L3.6mm_D1.6mm_P5.08mm_Horizontal" V 4130 1250 50  0001 C CNN
 F 3 "" H 4200 1250 50  0000 C CNN
 	1    4200 1250
@@
 F 0 "U6" H 5700 2100 50  0000 L CNN
 F 1 "TL074" H 5700 1700 50  0000 L CNN
-F 2 "" H 5650 2000 50  0000 C CNN
+F 2 "Housings_DIP:DIP-14_W7.62mm" H 5650 2000 50  0001 C CNN
 F 3 "" H 5750 2100 50  0000 C CNN
 	2    5700 1900
@@
 F 0 "R41" V 5330 2200 50  0000 C CNN
 F 1 "Rph" V 5250 2200 50  0000 C CNN
-F 2 "Resistors_ThroughHole:Resistor_Horizontal_RM7mm" V 5180 2200 50  0001 C CNN
+F 2 "scimpy_library:R_Axial_DIN0204_L3.6mm_D1.6mm_P5.08mm_Horizontal" V 5180 2200 50  0001 C CNN
 F 3 "" H 5250 2200 50  0000 C CNN
 	1    5250 2200
@@
 $EndComp
 $Comp
-L GND #PWR54
+L GND #PWR049
 U 1 1 590102C9
 P 5250 2350
-F 0 "#PWR54" H 5250 2100 50  0001 C CNN
+F 0 "#PWR049" H 5250 2100 50  0001 C CNN
 F 1 "GND" H 5250 2200 50  0000 C CNN
 F 2 "" H 5250 2350 50  0000 C CNN
@@
 F 0 "R39" V 5130 1150 50  0000 C CNN
 F 1 "2K2" V 5050 1150 50  0000 C CNN
-F 2 "Resistors_ThroughHole:Resistor_Horizontal_RM7mm" V 4980 1150 50  0001 C CNN
+F 2 "scimpy_library:R_Axial_DIN0204_L3.6mm_D1.6mm_P5.08mm_Horizontal" V 4980 1150 50  0001 C CNN
 F 3 "" H 5050 1150 50  0000 C CNN
 	1    5050 1150
@@
 F 0 "R40" V 5980 1150 50  0000 C CNN
 F 1 "2K2" V 5900 1150 50  0000 C CNN
-F 2 "Resistors_ThroughHole:Resistor_Horizontal_RM7mm" V 5830 1150 50  0001 C CNN
+F 2 "scimpy_library:R_Axial_DIN0204_L3.6mm_D1.6mm_P5.08mm_Horizontal" V 5830 1150 50  0001 C CNN
 F 3 "" H 5900 1150 50  0000 C CNN
 	1    5900 1150
@@
 F 0 "U6" H 4000 4100 50  0000 L CNN
 F 1 "TL074" H 4000 3700 50  0000 L CNN
-F 2 "" H 3950 4000 50  0000 C CNN
+F 2 "Housings_DIP:DIP-14_W7.62mm" H 3950 4000 50  0001 C CNN
 F 3 "" H 4050 4100 50  0000 C CNN
 	3    4000 3900
@@
 F 0 "R47" V 3630 4200 50  0000 C CNN
 F 1 "Rph" V 3550 4200 50  0000 C CNN
-F 2 "Resistors_ThroughHole:Resistor_Horizontal_RM7mm" V 3480 4200 50  0001 C CNN
+F 2 "scimpy_library:R_Axial_DIN0204_L3.6mm_D1.6mm_P5.08mm_Horizontal" V 3480 4200 50  0001 C CNN
 F 3 "" H 3550 4200 50  0000 C CNN
 	1    3550 4200
@@
 $EndComp
 $Comp
-L GND #PWR59
+L GND #PWR050
 U 1 1 59011086
 P 3550 4350
-F 0 "#PWR59" H 3550 4100 50  0001 C CNN
+F 0 "#PWR050" H 3550 4100 50  0001 C CNN
 F 1 "GND" H 3550 4200 50  0000 C CNN
 F 2 "" H 3550 4350 50  0000 C CNN
@@
 F 0 "R44" V 3430 3150 50  0000 C CNN
 F 1 "2K2" V 3350 3150 50  0000 C CNN
-F 2 "Resistors_ThroughHole:Resistor_Horizontal_RM7mm" V 3280 3150 50  0001 C CNN
+F 2 "scimpy_library:R_Axial_DIN0204_L3.6mm_D1.6mm_P5.08mm_Horizontal" V 3280 3150 50  0001 C CNN
 F 3 "" H 3350 3150 50  0000 C CNN
 	1    3350 3150
@@
 F 0 "R45" V 4280 3150 50  0000 C CNN
 F 1 "2K2" V 4200 3150 50  0000 C CNN
-F 2 "Resistors_ThroughHole:Resistor_Horizontal_RM7mm" V 4130 3150 50  0001 C CNN
+F 2 "scimpy_library:R_Axial_DIN0204_L3.6mm_D1.6mm_P5.08mm_Horizontal" V 4130 3150 50  0001 C CNN
 F 3 "" H 4200 3150 50  0000 C CNN
 	1    4200 3150
@@
 F 0 "U6" H 5700 4000 50  0000 L CNN
 F 1 "TL074" H 5700 3600 50  0000 L CNN
-F 2 "" H 5650 3900 50  0000 C CNN
+F 2 "Housings_DIP:DIP-14_W7.62mm" H 5650 3900 50  0001 C CNN
 F 3 "" H 5750 4000 50  0000 C CNN
 	4    5700 3800
@@
 F 0 "R46" V 5330 4100 50  0000 C CNN
 F 1 "Rph" V 5250 4100 50  0000 C CNN
-F 2 "Resistors_ThroughHole:Resistor_Horizontal_RM7mm" V 5180 4100 50  0001 C CNN
+F 2 "scimpy_library:R_Axial_DIN0204_L3.6mm_D1.6mm_P5.08mm_Horizontal" V 5180 4100 50  0001 C CNN
 F 3 "" H 5250 4100 50  0000 C CNN
 	1    5250 4100
@@
 $EndComp
 $Comp
-L GND #PWR58
+L GND #PWR051
 U 1 1 590110E0
 P 5250 4250
-F 0 "#PWR58" H 5250 4000 50  0001 C CNN
+F 0 "#PWR051" H 5250 4000 50  0001 C CNN
 F 1 "GND" H 5250 4100 50  0000 C CNN
 F 2 "" H 5250 4250 50  0000 C CNN
@@
 F 0 "R42" V 5130 3050 50  0000 C CNN
 F 1 "2K2" V 5050 3050 50  0000 C CNN
-F 2 "Resistors_ThroughHole:Resistor_Horizontal_RM7mm" V 4980 3050 50  0001 C CNN
+F 2 "scimpy_library:R_Axial_DIN0204_L3.6mm_D1.6mm_P5.08mm_Horizontal" V 4980 3050 50  0001 C CNN
 F 3 "" H 5050 3050 50  0000 C CNN
 	1    5050 3050
@@
 F 0 "R43" V 5980 3050 50  0000 C CNN
 F 1 "2K2" V 5900 3050 50  0000 C CNN
-F 2 "Resistors_ThroughHole:Resistor_Horizontal_RM7mm" V 5830 3050 50  0001 C CNN
+F 2 "scimpy_library:R_Axial_DIN0204_L3.6mm_D1.6mm_P5.08mm_Horizontal" V 5830 3050 50  0001 C CNN
 F 3 "" H 5900 3050 50  0000 C CNN
 	1    5900 3050
@@
 	5100 3900 5250 3900
 $Comp
-L GND #PWR53
+L GND #PWR052
 U 1 1 590200E6
 P 4100 1750
-F 0 "#PWR53" H 4100 1500 50  0001 C CNN
+F 0 "#PWR052" H 4100 1500 50  0001 C CNN
 F 1 "GND" H 4100 1600 50  0000 C CNN
 F 2 "" H 4100 1750 50  0000 C CNN
