File: boards/powersupply/powersupply.kicad_pcb (KiCad board)
At the start: 2 copper layers, 51.8 x 47 mm, 13 parts, among them P1 CONN_01X03, P2 CONN_01X03

Commit message: more boards work
Changed lines of the file:
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@@
   (general
     (links 17)
-    (no_connects 10)
-    (area 119.050999 21.514999 171.017001 68.655001)
+    (no_connects 1)
+    (area 113.070857 19.917 176.997143 70.61282)
     (thickness 1.6)
     (drawings 4)
@@
   (page A4)
   (layers
-    (0 F.Cu signal)
-    (31 B.Cu signal)
+    (0 F.Cu signal hide)
+    (31 B.Cu signal hide)
     (32 B.Adhes user)
     (33 F.Adhes user)
@@
     (descr "Mounting Hole 3.2mm, no annular, M3")
     (tags "mounting hole 3.2mm no annular m3")
-    (fp_text reference REF** (at 0 -4.2) (layer F.SilkS)
+    (fp_text reference REF** (at 0 -4.2) (layer F.SilkS) hide
       (effects (font (size 1 1) (thickness 0.15)))
     )
@@
     (descr "Radial Electrolytic Capacitor Diameter 22mm x Length 41mm, Pitch 10mm")
     (tags "Electrolytic Capacitor")
-    (fp_text reference C2 (at 5 -12.3 270) (layer F.SilkS)
+    (fp_text reference C2 (at -0.508 11.684 270) (layer F.SilkS)
       (effects (font (size 1 1) (thickness 0.15)))
     )
@@
     (descr "Single phase bridge rectifier case 18.5x5.5")
     (tags "Diode Bridge")
-    (fp_text reference D1 (at -2.1 -3.3 90) (layer F.SilkS)
+    (fp_text reference D1 (at 14.498 4.826 90) (layer F.SilkS)
       (effects (font (size 1 1) (thickness 0.15)))
     )
@@
     (descr "Capacitor 3mm Disc, Pitch 2.5mm")
     (tags Capacitor)
-    (fp_text reference C4 (at 1.25 -2.5 90) (layer F.SilkS)
+    (fp_text reference C4 (at -0.04 -2.286 90) (layer F.SilkS)
       (effects (font (size 1 1) (thickness 0.15)))
     )
@@
     (descr "Resistor, Axial, RM 15mm,")
     (tags "Resistor Axial RM 15mm")
-    (fp_text reference R3 (at 7.5 -3.74904 90) (layer F.SilkS)
+    (fp_text reference R3 (at 7.126 -2.286 90) (layer F.SilkS)
       (effects (font (size 1 1) (thickness 0.15)))
     )
@@
     (descr "Resistor, Axial, RM 15mm,")
     (tags "Resistor Axial RM 15mm")
-    (fp_text reference R2 (at 7.5 -3.74904 270) (layer F.SilkS)
+    (fp_text reference R2 (at 7.874 -2.54 270) (layer F.SilkS)
       (effects (font (size 1 1) (thickness 0.15)))
     )
@@
     (descr "Capacitor 3mm Disc, Pitch 2.5mm")
     (tags Capacitor)
-    (fp_text reference C1 (at 1.25 -2.5 90) (layer F.SilkS)
+    (fp_text reference C1 (at 2.246 -2.286 90) (layer F.SilkS)
       (effects (font (size 1 1) (thickness 0.15)))
     )
@@
     (at 150.93696 63.58382)
     (descr "3-way 5mm pitch terminal block, Phoenix MKDS series")
-    (fp_text reference P1 (at 5 5.9) (layer F.SilkS)
+    (fp_text reference P1 (at 13.90904 -4.40182 90) (layer F.SilkS)
       (effects (font (size 1 1) (thickness 0.15)))
     )
@@
     (at 160.782 27.432 180)
     (descr "3-way 5mm pitch terminal block, Phoenix MKDS series")
-    (fp_text reference P2 (at 5 5.9 180) (layer F.SilkS)
+    (fp_text reference P2 (at 13.716 3.302 270) (layer F.SilkS)
       (effects (font (size 1 1) (thickness 0.15)))
     )
@@
     (descr "Mounting Hole 3.2mm, no annular, M3")
     (tags "mounting hole 3.2mm no annular m3")
-    (fp_text reference REF** (at 0 -4.2) (layer F.SilkS)
+    (fp_text reference REF** (at 0 -4.2) (layer F.SilkS) hide
       (effects (font (size 1 1) (thickness 0.15)))
     )
@@
     (descr "Mounting Hole 3.2mm, no annular, M3")
     (tags "mounting hole 3.2mm no annular m3")
-    (fp_text reference REF** (at 0 -4.2) (layer F.SilkS)
+    (fp_text reference REF** (at 0 -4.2) (layer F.SilkS) hide
       (effects (font (size 1 1) (thickness 0.15)))
     )
@@
     (descr "Mounting Hole 3.2mm, no annular, M3")
     (tags "mounting hole 3.2mm no annular m3")
-    (fp_text reference REF** (at 0 -4.2) (layer F.SilkS)
-      (effects (font (size 1 1) (thickness 0.15)))
-    )
+    (fp_text reference REF** (at 0 -4.2) (layer F.SilkS) hide
+      (effects (font (size 1 1) (thickness 0.15)))
+    )
