File: boards/crossover/crossover.sch (KiCad schematic (older format))
At the start: 25 parts, among them P1 CONN_01X07, P2 CONN_01X07, U1 TL074

Commit message: board updates
Connections:
- net -15V: now also P1.2 (P2), P2.2 (P2); no longer P1.3 (P3), P2.3 (P3)
- net GND: now also P1.3 (P3), P2.3 (P3); no longer P1.2 (P2), P2.2 (P2)
- net right_low_out: now reaches C3.1, C4.1, P1.6 (P6), U1.6 (-), U1.7
- net right_high_out: now reaches P1.7 (P7), R1.2, U1.1, U1.2 (-)
- net left_low_out: now reaches C10.1, C11.1, P1.4 (P4), U1.13 (-), U1.14
- net left_high_out: now reaches P1.5 (P5), R6.2, U1.8, U1.9 (-)
Changed lines of the file:
@@
 	2150 1400 3150 1400
 Wire Wire Line
-	2150 1400 2150 2650
+	2150 2650 2150 1400
 Wire Wire Line
 	2450 4050 2450 2850
@@
 L GND #PWR07
 U 1 1 590EE231
-P 1400 3150
-F 0 "#PWR07" H 1400 2900 50  0001 C CNN
-F 1 "GND" H 1400 3000 50  0000 C CNN
-F 2 "" H 1400 3150 50  0000 C CNN
-F 3 "" H 1400 3150 50  0000 C CNN
-	1    1400 3150
+P 1550 3050
+F 0 "#PWR07" H 1550 2800 50  0001 C CNN
+F 1 "GND" H 1550 2900 50  0000 C CNN
+F 2 "" H 1550 3050 50  0000 C CNN
+F 3 "" H 1550 3050 50  0000 C CNN
+	1    1550 3050
 	1    0    0    -1
 $EndComp
@@
 $EndComp
 $Comp
-L -15V #PWR6
+L -15V #PWR8
 U 1 1 590EE75F
-P 1550 3050
-F 0 "#PWR6" H 1550 3150 50  0001 C CNN
-F 1 "-15V" H 1550 3200 50  0000 C CNN
-F 2 "" H 1550 3050 50  0000 C CNN
-F 3 "" H 1550 3050 50  0000 C CNN
-	1    1550 3050
+P 1400 3150
+F 0 "#PWR8" H 1400 3250 50  0001 C CNN
+F 1 "-15V" H 1400 3300 50  0000 C CNN
+F 2 "" H 1400 3150 50  0000 C CNN
+F 3 "" H 1400 3150 50  0000 C CNN
+	1    1400 3150
 	-1   0    0    1
 $EndComp
@@
 L GND #PWR010
 U 1 1 590F0B02
-P 6650 3050
-F 0 "#PWR010" H 6650 2800 50  0001 C CNN
-F 1 "GND" H 6650 2900 50  0000 C CNN
-F 2 "" H 6650 3050 50  0000 C CNN
-F 3 "" H 6650 3050 50  0000 C CNN
-	1    6650 3050
+P 6500 2950
+F 0 "#PWR010" H 6500 2700 50  0001 C CNN
+F 1 "GND" H 6500 2800 50  0000 C CNN
+F 2 "" H 6500 2950 50  0000 C CNN
+F 3 "" H 6500 2950 50  0000 C CNN
+	1    6500 2950
 	-1   0    0    -1
 $EndComp
@@
 $EndComp
 $Comp
-L -15V #PWR5
+L -15V #PWR7
 U 1 1 590F0B11
-P 6500 2950
-F 0 "#PWR5" H 6500 3050 50  0001 C CNN
-F 1 "-15V" H 6500 3100 50  0000 C CNN
-F 2 "" H 6500 2950 50  0000 C CNN
-F 3 "" H 6500 2950 50  0000 C CNN
-	1    6500 2950
+P 6650 3050
+F 0 "#PWR7" H 6650 3150 50  0001 C CNN
+F 1 "-15V" H 6650 3200 50  0000 C CNN
+F 2 "" H 6650 3050 50  0000 C CNN
+F 3 "" H 6650 3050 50  0000 C CNN
+	1    6650 3050
 	1    0    0    1
 $EndComp
@@
 Text Notes 6700 4400 0    60   ~ 0
 single stage filter\n
+Text Label 5400 1500 0    60   ~ 0
+right_high_out
+Text Label 5300 2750 0    60   ~ 0
+right_low_out
+Text Label 5300 4150 0    60   ~ 0
+left_high_out
+Text Label 5350 5400 0    60   ~ 0
+left_low_out
 $EndSCHEMATC
